File: g030f6.brd (EAGLE design)
At the start: 100 x 80 mm, 40 parts, among them IC1 24LC128SM, U1 AMS1117

Commit message: checked, TODO minimize size
Parts:
- moved C13 5.57 mm to (39.8, 31.5), turned to 180 degrees
- moved R11 3.07 mm to (40.2, 51.9), turned to 180 degrees
- moved C11 2.85 mm to (39.1, 59.6), turned to 180 degrees
- moved R14 2.70 mm to (37.7, 62.3)
- moved R15 2.68 mm to (37.7, 63.3)
- moved U1 2.26 mm to (42.6, 57.0)
- moved LED1 1.98 mm to (35.6, 62.3), turned to 0 degrees
- moved R5 1.47 mm to (37.2, 41.1)
- moved C7 1.36 mm to (35.6, 65.8)
- moved LED2 1.36 mm to (35.6, 63.3), turned to 0 degrees
- moved C2 0.91 mm to (38.1, 44.7)
- moved C9 0.71 mm to (37.7, 65.9)
- moved C6 0.68 mm to (40.7, 52.6)
- moved R2 0.64 mm to (48.3, 63.8)
- moved C10 0.62 mm to (48.3, 59.7)
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Routing:
- net N$4: track 12.4 -> 21.4 mm, vias 0 -> 2
- net N$30: track 26.3 -> 34.2 mm
- net GND: track 37.5 -> 45.4 mm, vias 13 -> 16
- net +3V3: track 68.4 -> 61.6 mm
- net N$25: track 39.2 -> 35.4 mm, vias 3 -> 2
- net N$26: track 39.0 -> 35.2 mm, vias 3 -> 2
- net N$36: track 8.57 -> 6.78 mm
- net N$19: track 6.45 -> 4.71 mm
- net N$7: track 7.21 -> 5.52 mm
- net +5V: track 30.3 -> 28.6 mm
- net N$1: track 3.97 -> 5.43 mm
- net N$11: track 1.76 -> 0.88 mm
- net N$8: track 14.8 -> 15.6 mm
- net N$12: track 1.47 -> 0.86 mm
